Commit message: Further work on force transformation.

File: urdf2casadi/examples/urdf/ur5_mod.urdf (robot description, URDF)
Before this commit: robot ur5, 8 links, 7 joints
Links:
- added link force_plate, mass 36.0
Joints:
- added joint force_plate__base_link: type fixed, parent force_plate, child base_link, origin xyz=0.0 0.0 0.0 rpy=0.0 0.0 0.0
