Commit message: Use dummy elements in urdf for force plate data transformation into first joint.

File: Scripts/Common/ur5_mod.urdf (robot description, URDF)
Before this commit: robot ur5, 9 links, 8 joints
Links:
- removed link force_plate
- added link dummy_link, mass 100.0
Joints:
- removed joint force_plate__base_link
- added joint dummy_joint: type revolute, parent dummy_link, child base_link, origin xyz=0.0 0.0 0.089159 rpy=0.0 0.0 0.0, axis 0 0 1, limit lower=-6.28318530718 upper=6.28318530718 effort=150.0 velocity=3.15
