Commit message: Use another urdf file, fixed transformation, ...

File: Scripts/Common/ur5e.urdf (robot description, URDF)
Before this commit: robot ur5e_robot, 11 links, 10 joints
Links:
- removed link base
- link tool0: mass None -> 0.6
Joints:
- removed joint base_link-base_fixed_joint
- joint base_link-base_link_inertia: axis (none) -> 0 0 1; type fixed -> revolute
